Commit message: added base_footprint link

File: racecar_description/urdf/racecar.xacro (robot description, xacro)
@@ -3,5 +3,11 @@
   <xacro:include filename="$(find racecar_description)/urdf/macros.xacro" />
   <!-- Add chassis and it's inertia link -->
-  <link name="base_link" />
+  <link name="base_footprint"></link>
+  <link name="base_link"></link>
+  <joint name="base_footprint_joint" type="fixed">
+    <origin xyz="-0.1625 0 0" rpy="0 0 0" />
+    <parent link="base_footprint"/>
+    <child link="base_link" />
+  </joint>
   <link name="chassis">
     <visual>

Commit message: Added .rviz

File: racecar_description/urdf/racecar.xacro (robot description, xacro)
@@ -6,5 +6,5 @@
   <link name="base_link"></link>
   <joint name="base_footprint_joint" type="fixed">
-    <origin xyz="-0.1625 0 0" rpy="0 0 0" />
+    <origin xyz="-0.325 0 0" rpy="0 0 0" />
     <parent link="base_footprint"/>
     <child link="base_link" />
